File: beryl_rain.kicad_pcb (KiCad board)
At the start: 2 copper layers, 26.7 x 49.5 mm, 18 parts, among them CON1 POWER, P1 POWER, P2 FTDI, P3 IR, P4 RESET, P5 PROG, SW1 SWITCH, U1 NCP1117ST33T3G, U2 ESP-12

Commit message: Completed version 1
Parts:
- CON1: footprint Connect:BARREL_JACK -> timhawes:BARREL_JACK
- moved C5 0.34 mm to (145.2, 103.1), turned to 90 degrees
Connections:
- U1 pad 4: (no net) -> +3V3
Routing:
- net +3V3: track 47.5 -> 55.0 mm
- net GND: track 96.6 -> 97.7 mm
- net +5V: track 43.1 -> 42.6 mm
- added copper zone on F.Cu, net +3V3
